Commit message: latest code after changing to landmark based slam

File: src/autonomous_exploration/urdf/turtlebot3_waffle_pi.urdf (robot description, URDF)
Before this commit: robot turtlebot3_waffle_pi, 11 links, 10 joints
Links:
- link ${namespace}base_link: geometry collision box size=0.266 0.266 0.094; visual mesh filename=package://autonomous_exploration/meshes/bases/waffle_pi_bas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 scale=0.001 0.001 0.001
- link ${namespace}base_scan: geometry collision cylinder length=0.0315 radius=0.055; visual mesh filename=package://autonomous_exploration/meshes/sensors/lds.stl scale=0.001 0.001 0.001
- link ${namespace}wheel_left_link: geometry collision cylinder length=0.018 radius=0.033; visual mesh filename=package://autonomous_exploration/meshes/wheels/left_tire.stl scale=0.001 0.001 0.001
- link ${namespace}wheel_right_link: geometry collision cylinder length=0.018 radius=0.033; visual mesh filename=package://autonomous_exploration/meshes/wheels/right_tire.s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 scale=0.001 0.001 0.001
